File: cad/iwr6843_spi_adapter/iwr6843_spi_adapter.kicad_sch (KiCad schematic)
At the start: 15 parts, among them J1 QTH-030-01-L-D-A, J2 Pi5_jumpers, U1 SN74LVC2G34DBVR, U2 SN74LVC2G34DBVR, U3 SN74LVC2G34DBVR

Commit message: feat(cad): PCBWay turnkey BOM/CPL, assembly drawings, export_fab.sh
Real MPNs and manufacturers for all assembled parts (single source in
generate.py), PCBWay-format BOM, CPL without the hand-soldered J2
header, scaled assembly drawings with pad numbers, and export_fab.sh
that regenerates and refuses to export on any ERC/DRC error.

Co-Authored-By: Claude Opus 5.5 <noreply@anthropic.com>
Parts:
- C1, C2, C3: MPN 0603 X7R 100nF 16V -> CL10B104KB8NNNC
- J2: MPN 2.54mm 1x11 pin header -> (none)
- R1, R2, R3, R4, R5: MPN 0603 1% 100k -> RC0603FR-07100KL
- R6, R7: MPN 0603 1% 33R -> RC0603FR-0733RL
Changed lines of the file:
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@@
 		(property "Footprint" "Connector_PinHeader_2.54mm:PinHeader_1x11_P2.54mm_Vertical" (at 254.00 76.20 0) (effects (font (size 1.27 1.27)) (hide yes)))
 		(property "Datasheet" "" (at 254.00 76.20 0) (effects (font (size 1.27 1.27)) (hide yes)))
-		(property "MPN" "2.54mm 1x11 pin header" (at 254.00 76.20 0) (effects (font (size 1.27 1.27)) (hide yes)))
+		(property "MPN" "" (at 254.00 76.20 0) (effects (font (size 1.27 1.27)) (hide yes)))
 		(pin "1")
 		(pin "2")
@@
 		(property "Footprint" "Capacitor_SMD:C_0603_1608Metric" (at 132.08 172.72 0) (effects (font (size 1.27 1.27)) (hide yes)))
 		(property "Datasheet" "" (at 132.08 172.72 0) (effects (font (size 1.27 1.27)) (hide yes)))
-		(property "MPN" "0603 X7R 100nF 16V" (at 132.08 172.72 0) (effects (font (size 1.27 1.27)) (hide yes)))
+		(property "MPN" "CL10B104KB8NNNC" (at 132.08 172.72 0) (effects (font (size 1.27 1.27)) (hide yes)))
 		(pin "1")
 		(pin "2")
@@
 		(property "Footprint" "Capacitor_SMD:C_0603_1608Metric" (at 142.24 172.72 0) (effects (font (size 1.27 1.27)) (hide yes)))
 		(property "Datasheet" "" (at 142.24 172.72 0) (effects (font (size 1.27 1.27)) (hide yes)))
-		(property "MPN" "0603 X7R 100nF 16V" (at 142.24 172.72 0) (effects (font (size 1.27 1.27)) (hide yes)))
+		(property "MPN" "CL10B104KB8NNNC" (at 142.24 172.72 0) (effects (font (size 1.27 1.27)) (hide yes)))
 		(pin "1")
 		(pin "2")
@@
 		(property "Footprint" "Capacitor_SMD:C_0603_1608Metric" (at 152.40 172.72 0) (effects (font (size 1.27 1.27)) (hide yes)))
 		(property "Datasheet" "" (at 152.40 172.72 0) (effects (font (size 1.27 1.27)) (hide yes)))
-		(property "MPN" "0603 X7R 100nF 16V" (at 152.40 172.72 0) (effects (font (size 1.27 1.27)) (hide yes)))
+		(property "MPN" "CL10B104KB8NNNC" (at 152.40 172.72 0) (effects (font (size 1.27 1.27)) (hide yes)))
 		(pin "1")
 		(pin "2")
@@
 		(property "Footprint" "Resistor_SMD:R_0603_1608Metric" (at 203.20 101.60 0) (effects (font (size 1.27 1.27)) (hide yes)))
 		(property "Datasheet" "" (at 203.20 101.60 0) (effects (font (size 1.27 1.27)) (hide yes)))
-		(property "MPN" "0603 1% 100k" (at 203.20 101.60 0) (effects (font (size 1.27 1.27)) (hide yes)))
+		(property "MPN" "RC0603FR-07100KL" (at 203.20 101.60 0) (effects (font (size 1.27 1.27)) (hide yes)))
 		(pin "1")
 		(pin "2")
@@
 		(property "Footprint" "Resistor_SMD:R_0603_1608Metric" (at 203.20 60.96 0) (effects (font (size 1.27 1.27)) (hide yes)))
 		(property "Datasheet" "" (at 203.20 60.96 0) (effects (font (size 1.27 1.27)) (hide yes)))
-		(property "MPN" "0603 1% 100k" (at 203.20 60.96 0) (effects (font (size 1.27 1.27)) (hide yes)))
+		(property "MPN" "RC0603FR-07100KL" (at 203.20 60.96 0) (effects (font (size 1.27 1.27)) (hide yes)))
 		(pin "1")
 		(pin "2")
@@
 		(property "Footprint" "Resistor_SMD:R_0603_1608Metric" (at 203.20 45.72 0) (effects (font (size 1.27 1.27)) (hide yes)))
 		(property "Datasheet" "" (at 203.20 45.72 0) (effects (font (size 1.27 1.27)) (hide yes)))
-		(property "MPN" "0603 1% 100k" (at 203.20 45.72 0) (effects (font (size 1.27 1.27)) (hide yes)))
+		(property "MPN" "RC0603FR-07100KL" (at 203.20 45.72 0) (effects (font (size 1.27 1.27)) (hide yes)))
 		(pin "1")
 		(pin "2")
@@
 		(property "Footprint" "Resistor_SMD:R_0603_1608Metric" (at 119.38 147.32 0) (effects (font (size 1.27 1.27)) (hide yes)))
 		(property "Datasheet" "" (at 119.38 147.32 0) (effects (font (size 1.27 1.27)) (hide yes)))
-		(property "MPN" "0603 1% 100k" (at 119.38 147.32 0) (effects (font (size 1.27 1.27)) (hide yes)))
+		(property "MPN" "RC0603FR-07100KL" (at 119.38 147.32 0) (effects (font (size 1.27 1.27)) (hide yes)))
 		(pin "1")
 		(pin "2")
@@
 		(property "Footprint" "Resistor_SMD:R_0603_1608Metric" (at 119.38 132.08 0) (effects (font (size 1.27 1.27)) (hide yes)))
 		(property "Datasheet" "" (at 119.38 132.08 0) (effects (font (size 1.27 1.27)) (hide yes)))
-		(property "MPN" "0603 1% 100k" (at 119.38 132.08 0) (effects (font (size 1.27 1.27)) (hide yes)))
+		(property "MPN" "RC0603FR-07100KL" (at 119.38 132.08 0) (effects (font (size 1.27 1.27)) (hide yes)))
 		(pin "1")
 		(pin "2")
@@
 		(property "Footprint" "Resistor_SMD:R_0603_1608Metric" (at 203.20 132.08 0) (effects (font (size 1.27 1.27)) (hide yes)))
 		(property "Datasheet" "" (at 203.20 132.08 0) (effects (font (size 1.27 1.27)) (hide yes)))
-		(property "MPN" "0603 1% 33R" (at 203.20 132.08 0) (effects (font (size 1.27 1.27)) (hide yes)))
+		(property "MPN" "RC0603FR-0733RL" (at 203.20 132.08 0) (effects (font (size 1.27 1.27)) (hide yes)))
 		(pin "1")
 		(pin "2")
@@
 		(property "Footprint" "Resistor_SMD:R_0603_1608Metric" (at 203.20 147.32 0) (effects (font (size 1.27 1.27)) (hide yes)))
 		(property "Datasheet" "" (at 203.20 147.32 0) (effects (font (size 1.27 1.27)) (hide yes)))
-		(property "MPN" "0603 1% 33R" (at 203.20 147.32 0) (effects (font (size 1.27 1.27)) (hide yes)))
-		(pin "1")
-		(pin "2")
+		(property "MPN" "RC0603FR-0733RL" (at 203.20 147.32 0) (effects (font (size 1.27 1.27)) (hide yes)))
+		(pin "1")
+		(pin "2")
